Commit message: Lab 2 Commit 2
This is the second commit for lab 2, which fixes all issues from previous commit and finishes lab 2.

File: urdf/lab2nav.urdf (robot description, URDF)
Before this commit: robot navvis, 8 links, 7 joints
Links:
- removed link wheel_center
- removed link wheel_right
- link base: geometry collision box size=0.45 0.78 1.98; visual box size=0.45 0.78 1.98
Joints:
- removed joint base_wheel_center_joint
- removed joint base_wheel_right_joint

File: urdf/nav2.xacro (robot description, xacro)
@@ -1,5 +1,4 @@
 <?xml version="1.0"?>
 <robot xmlns:xacro="http://www.ros.org/wiki/xacro" name="navvis">
-<robot name="navvis">
 <link name="base">
 <visual>
@@ -7,5 +6,5 @@
 <origin xyz="0.0 0.0 0.96" rpy="0.0 0.0 0.0" />
 <geometry>
-<box size="0.45 0.78 1.92" />
+<box size="0.45 0.78 1.98" />
 </geometry>
 </visual>
@@ -14,12 +13,12 @@
 <origin xyz="0.0 0.0 0.96" rpy="0.0 0.0 0.0" />
 <geometry>
-<box size="0.45 0.78 1.92" />
+<box size="0.45 0.78 1.98" />
 </geometry>
 </collision>
 </link>
+<!--
 <link name="laser_vert_bottom">
 <visual>
-<!-- Shift the box up half its height. !-->
-<origin xyz="0.3158 -0.0021 0.5100" rpy="3.1355 -1.3045 0.0025" />
+<origin xyz="0.0 0.0 0.0435" rpy="0.0 0.0 0.0" />
 <geometry>
 <box size="0.062 0.062 0.087" />
@@ -27,6 +26,5 @@
 </visual>
 <collision>
-<!-- Shift the box up half its height. !-->
-<origin xyz="0.3158 -0.0021 0.5100" rpy="3.1355 -1.3045 0.0025" />
+<origin xyz="0.0 0.0 0.0435" rpy="0.0 0.0 0.0" />
 <geometry>
 <box size="0.062 0.062 0.087" />
@@ -36,6 +34,5 @@
 <link name="laser_vert_top_right">
 <visual>
-<!-- Shift the box up half its height. !-->
-<origin xyz="0.2978 -0.1450 1.8451" rpy="-1.1760 0.6313 -1.9377" />
+<origin xyz="0.0 0.0 0.0435" rpy="0.0 0.0 0.0" />
 <geometry>
 <box size="0.062 0.062 0.087" />
@@ -43,6 +40,5 @@
 </visual>
 <collision>
-<!-- Shift the box up half its height. !-->
-<origin xyz="0.2978 -0.1450 1.8451" rpy="-1.1760 0.6313 -1.9377" />
+<origin xyz="0.0 0.0 0.0435" rpy="0.0 0.0 0.0" />
 <geometry>
 <box size="0.062 0.062 0.087" />
@@ -52,6 +48,5 @@
 <link name="laser_vert_top_left">
 <visual>
-<!-- Shift the box up half its height. !-->
-<origin xyz="0.2997 0.1531 1.8443" rpy="1.1780 0.6198 1.9560" />
+<origin xyz="0.0 0.0 0.0435" rpy="0.0 0.0 0.0" />
 <geometry>
 <box size="0.062 0.062 0.087" />
@@ -59,6 +54,5 @@
 </visual>
 <collision>
-<!-- Shift the box up half its height. !-->
-<origin xyz="0.2997 0.1531 1.8443" rpy="1.1780 0.6198 1.9560" />
+<origin xyz="0.0 0.0 0.0435" rpy="0.0 0.0 0.0" />
 <geometry>
 <box size="0.062 0.062 0.087" />
@@ -68,5 +62,5 @@
 <link name="laser_horiz">
 <visual>
-<origin xyz="0.2325 0.0001 1.9201" rpy="-0.0012 0.1146 -0.0015" />
+<origin xyz="0.0 0.0 0.026" rpy="0.0 0.0 0.0" />
 <geometry>
 <cylinder radius="0.052" length="0.072"/>
@@ -74,5 +68,5 @@
 </visual>
 <collision>
-<origin xyz="0.2325 0.0001 1.9201" rpy="-0.0012 0.1146 -0.0015" />
+<origin xyz="0.0 0.0 0.026" rpy="0.0 0.0 0.0" />
 <geometry>
 <cylinder radius="0.052" length="0.072"/>
@@ -80,4 +74,18 @@
 </collision>
 </link>
+!-->
+<!-- Include the XACRO file that defines a Hokuyo LIDAR. -->
+<xacro:include filename="$(find gazebo_plugins)/test/multi_robot_scenario/xacro/laser/hokuyo.xacro" />
+<xacro:laser name="laser_vert_bottom" parent="base" xyz="0.3158 -0.0021 0.5100" rpy="3.1355 -1.3045 0.0025" meshes="package://gazebo_plugins/test/multi_robot_scenario/meshes/laser" />
+<xacro:laser name="laser_vert_top_right" parent="base" xyz="0.2978 -0.1450 1.8451" rpy="-1.1760 0.6313 -1.9377" meshes="package://gazebo_plugins/test/multi_robot_scenario/meshes/laser" />
+<xacro:laser name="laser_vert_top_left" parent="base" xyz="0.2997 0.1531 1.8443" rpy="1.1780 0.6198 1.9560" meshes="package://gazebo_plugins/test/multi_robot_scenario/meshes/laser" />
+<xacro:include filename="$(find velodyne_description)/urdf/VLP-16.urdf.xacro"/>
+<!-- Invoke the macro to define the Hokuyo LIDAR. -->
+<xacro:VLP-16 parent="base" name="laser_horiz" topic="laser_horiz/packets" hz="10"
+samples="440" gpu="false">
+<origin xyz="0.2325416305773505 -0.0001380069427607134 1.920122926231907"
+rpy="-0.0012068 0.114646 -0.0015308" />
+</xacro:VLP-16>
+<!--
 <joint name="base_laser_vert_bottom_joint" type="fixed">
 <parent link="base" />
@@ -100,9 +108,10 @@
 <origin xyz="0.2325 0.0001 1.9201" rpy="-0.0012 0.1146 -0.0015" />
 </joint>
+!-->
 <!-- XACRO Macro definition block to add around the wheel link and joint !-->
-<xacro:macro name="xacro_name" params="side reflect">
-	<link name="wheel_left">
+<xacro:macro name="side_wheels" params="side reflect">
+	<link name="wheel_${side}">
 	<visual>
-	<origin xyz="-0.1 0.4 0.0" rpy="-1.570 0.0 0.0" />
+	<origin xyz="0.0 0.0 0.0" rpy="0.0 0.0 0.0" />
 	<geometry>
 	<cylinder radius="0.2" length="0.05"/>
@@ -110,5 +119,5 @@
 	</visual>
 	<collision>
-	<origin xyz="-0.1 0.4 0.0" rpy="-1.570 0.0 0.0" />
+	<origin xyz="0.0 0.0 0.0" rpy="0.0 0.0 0.0" />
 	<geometry>
 	<cylinder radius="0.2" length="0.05"/>
@@ -116,41 +125,19 @@
 	</collision>
 	</link>
-	<joint name="base_wheel_left_joint" type="fixed">
+	<joint name="base_wheel_${side}_joint" type="continuous">
 	<parent link="base" />
-	<child link="wheel_left" />
-	<origin xyz="-0.1 0.4 0.0" rpy="-1.570 0.0 0.0" />
+	<child link="wheel_${side}" />
+	<origin xyz="-0.10 ${reflect * 0.4} 0.0" rpy="-1.570 0.0 0.0" />
+	<axis xyz = "0.0 0.0 1.0" />
+	<limit effort = "100" velocity = "100" />
 	</joint>
 </xacro:macro>
 <!-- Call the XACRO Macro.  It should be the left wheel !-->
-<xacro:xacro_name side="left" reflect="1" />
-<!-- XACRO Macro definition block to add around the wheel link and joint !-->
-<xacro:macro name="xacro_name" params="side reflect">
-	<link name="wheel_right">
-	<visual>
-	<origin xyz="-0.1 0.4 0.0" rpy="-1.570 0.0 0.0" />
-	<geometry>
-	<cylinder radius="0.2" length="0.05"/>
-	</geometry>
-	</visual>
-	<collision>
-	<origin xyz="-0.1 0.4 0.0" rpy="-1.570 0.0 0.0" />
-	<geometry>
-	<cylinder radius="0.2" length="0.05"/>
-	</geometry>
-	</collision>
-	</link>
-	<joint name="base_wheel_right_joint" type="fixed">
-	<parent link="base" />
-	<child link="wheel_right" />
-	<origin xyz="-0.1 0.4 0.0" rpy="-1.570 0.0 0.0" />
-	</joint>
-</xacro:macro>
-<!-- Call the XACRO Macro.  It should be the left wheel !-->
-<xacro:xacro_name side="right" reflect="-1" />
-<!-- XACRO Macro definition block to add around the wheel link and joint !-->
-<xacro:macro name="xacro_name" params="side reflect">
+<xacro:side_wheels side="left" reflect="1" />
+<xacro:side_wheels side="right" reflect="-1" />
+<xacro:macro name="center">
 	<link name="wheel_center">
 	<visual>
-	<origin xyz="0.1 0.0 0.0" rpy="-1.570 0.0 0.0" />
+	<origin xyz="0.0 0.0 0.0" rpy="0.0 0.0 0.0" />
 	<geometry>
 	<cylinder radius="0.15" length="0.05"/>
@@ -158,5 +145,5 @@
 	</visual>
 	<collision>
-	<origin xyz="0.1 0.0 0.0" rpy="-1.570 0.0 0.0" />
+	<origin xyz="0.0 0.0 0.0" rpy="0.0 0.0 0.0" />
 	<geometry>
 	<cylinder radius="0.15" length="0.05"/>
@@ -164,11 +151,12 @@
 	</collision>
 	</link>
-	<joint name="base_wheel_center_joint" type="fixed">
+	<joint name="base_wheel_center_joint" type="continuous">
 	<parent link="base" />
 	<child link="wheel_center" />
-	<origin xyz="0.1 0.0 0.0" rpy="-1.570 0.0 0.0" />
+	<origin xyz="0.1 0.0 -0.025" rpy="-1.570 0.0 0.0" />
+	<axis xyz = "0.0 0.0 1.0" />
+	<limit effort = "100" velocity = "100" />
 	</joint>
 </xacro:macro>
-<!-- Call the XACRO Macro.  It should be the left wheel !-->
-<xacro:xacro_name side="left" reflect="1" />
+<xacro:center />
 </robot>
